File: plant led.kicad_pcb (KiCad board)
At the start: 2 copper layers, 80 x 80 mm, 38 parts, among them J1 Conn_01x01_Pin, J2 Conn_01x01_Pin, M3 MountingHole_3.2mm_M3_DIN965, M5 MountingHole_5.3mm_M5_DIN965

Commit message: feat(pcb): add v1.0.3 silkscreen guides
  Add silkscreen rings around the mounting and cable holes.
  Document the current MCPCB design, project status, and preview images.
Other:
- board text added: "Grow light v1.0.3 2026-07-27"
- board text removed: "Grow light v1.0.2 2026-07-11"
Changed lines of the file:
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@@
 		(capping no)
 		(filling no)
-		(zone_defaults)
 		(pcbplotparams
 			(layerselection 0x00000000_00000000_55555555_57555573)
@@
 		(tags "mountinghole M5 DIN965")
 		(property "Reference" "M5"
-			(at 0 -5.55 0)
+			(at 0 -5.75 0)
 			(layer "F.SilkS")
 			(effects
@@
 		(layer "F.SilkS")
 	)
+	(gr_circle
+		(center 129.076756 106.798374)
+		(end 132.076756 106.798374)
+		(stroke
+			(width 0.2)
+			(type default)
+		)
+		(fill no)
+		(layer "F.SilkS")
+	)
+	(gr_circle
+		(center 133.650813 85.279127)
+		(end 136.650813 85.279127)
+		(stroke
+			(width 0.2)
+			(type default)
+		)
+		(fill no)
+		(layer "F.SilkS")
+	)
+	(gr_circle
+		(center 145.425943 121.519248)
+		(end 148.425943 121.519248)
+		(stroke
+			(width 0.2)
+			(type default)
+		)
+		(fill no)
+		(layer "F.SilkS")
+	)
+	(gr_circle
+		(center 150 100)
+		(end 155 100)
+		(stroke
+			(width 0.2)
+			(type default)
+		)
+		(fill no)
+		(layer "F.SilkS")
+	)
+	(gr_circle
+		(center 154.574057 78.480752)
+		(end 157.574057 78.480752)
+		(stroke
+			(width 0.2)
+			(type default)
+		)
+		(fill no)
+		(layer "F.SilkS")
+	)
+	(gr_circle
+		(center 166.349186 114.720873)
+		(end 169.349186 114.720873)
+		(stroke
+			(width 0.2)
+			(type default)
+		)
+		(fill no)
+		(layer "F.SilkS")
+	)
 	(gr_rect
 		(start 169.3 104.2)
@@
 		(layer "F.SilkS")
 	)
+	(gr_circle
+		(center 170.923244 93.201626)
+		(end 173.923244 93.201626)
+		(stroke
+			(width 0.2)
+			(type default)
+		)
+		(fill no)
+		(layer "F.SilkS")
+	)
 	(gr_line
 		(start 137.63932 61.957739)
@@
 		(layer "Edge.Cuts")
 	)
-	(gr_text "Grow light\nv1.0.2 2026-07-11"
-		(at 133.6 100.7 0)
+	(gr_text "Grow light\nv1.0.3 2026-07-27"
+		(at 133.2 100.7 0)
 		(layer "F.SilkS")
 		(effects

Commit message: feat(pcb): add power polarity silkscreen labels
Other:
- board text added: "+"
- board text added: "-"
Changed lines of the file:
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@@
 		(layer "Edge.Cuts")
+	)
+	(gr_text "-"
+		(at 144.5 95.1 0)
+		(layer "F.SilkS")
+		(effects
+			(font
+				(size 1.5 1.5)
+				(thickness 0.3)
+				(bold yes)
+			)
+			(justify left bottom)
+		)
+	)
+	(gr_text "+"
+		(at 153.3 95.3 0)
+		(layer "F.SilkS")
+		(effects
+			(font
+				(size 1.5 1.5)
+				(thickness 0.3)
+				(bold yes)
+			)
+			(justify left bottom)
+		)
 	)
 	(gr_text "Grow light\nv1.0.3 2026-07-27"
